Commit message: added more scenarios

File: urdf/roahm/mug.xacro (robot description, xacro)
@@ -14,4 +14,8 @@
         <geometry>
           <mesh filename="package://franka_description/meshes/mug.dae"/>
+          <!-- <mesh filename="file:///home/sid/.julia/dev/PBDS/urdf/meshes/mug.dae"/>  -->
+          <!--/// means absolute path-->
+          <!-- <mesh filename="file://../meshes/mug.dae"/> -->
+          <!-- <mesh filename="package://$(find panda_roahm)/worlds/mug.dae"/> -->
         </geometry>
       </visual>
