Commit message: fixed rotated base_link issue; added more scenarios

File: urdf/roahm/mug_panda_arm_hand_fingers_fixed.urdf (robot description, URDF)
Before this commit: robot panda, 15 links, 14 joints
Joints:
- joint mug_joint: origin xyz=0.5 0.5 0 rpy=0 0 0 -> xyz=0.5 0.5 0.5 rpy=0 0 0

File: urdf/roahm/mug_panda_arm_hand_fingers_fixed.urdf.xacro (robot description, xacro)
@@ -6,4 +6,5 @@
   <xacro:hand_fingers_fixed ns="panda" rpy="0 0 ${-pi/4}" connected_to="panda_link8" q_fingers="0.02"/>
   <xacro:include filename="mug.xacro"/>
-  <xacro:mug connected_to="panda_link0" xyz="0.5 0.5 0"/>
+  <!-- <xacro:mug connected_to="panda_link0" xyz="0.5 0.5 0"/> -->
+  <xacro:mug connected_to="panda_link0" xyz="0.5 0.5 0.5"/>
 </robot>

File: urdf/roahm/panda_arm.xacro (robot description, xacro)
@@ -1,6 +1,5 @@
 <?xml version='1.0' encoding='utf-8'?>
 <robot xmlns:xacro="http://www.ros.org/wiki/xacro" name="panda">
-  <!-- <xacro:macro name="panda_arm" params="arm_id:='panda' description_pkg:='franka_description' connected_to:='' xyz:='0 0 0' rpy:='0 0 0'"> -->
-  <xacro:macro name="panda_arm" params="arm_id:='panda' description_pkg:='franka_description' connected_to:='' xyz:='0 0 0' rpy:='${-pi/2} 0 0'">
+  <xacro:macro name="panda_arm" params="arm_id:='panda' description_pkg:='franka_description' connected_to:='' xyz:='0 0 0' rpy:='0 0 0'">
     <xacro:unless value="${not connected_to}">
       <joint name="${arm_id}_joint_${connected_to}" type="fixed">
@@ -37,5 +36,4 @@
       <safety_controller k_position="100.0" k_velocity="40.0" soft_lower_limit="-2.8973" soft_upper_limit="2.8973"/>
       <origin rpy="0 0 0" xyz="0 0 0.333"/>
-      <!-- <origin rpy="0 0 ${-pi/2}" xyz="0 0 0.333"/> -->
       <parent link="${arm_id}_link0"/>
       <child link="${arm_id}_link1"/>

File: urdf/roahm/sphere_col/table_mug_panda_arm_hand_fingers_fixed.urdf (robot description, URDF)
Before this commit: robot panda, 16 links, 15 joints
Joints:
- joint panda_joint_table: origin xyz=0 0 0 rpy=0 0 1.57079632679 -> xyz=0 0 0 rpy=0 0 0

File: urdf/roahm/sphere_col/table_mug_panda_arm_hand_fingers_fixed.urdf.xacro (robot description, xacro)
@@ -5,5 +5,6 @@
   <xacro:include filename="panda_arm.xacro"/>
   <xacro:include filename="hand_fingers_fixed.xacro"/>
-  <xacro:panda_arm connected_to="table" xyz="${pandax} ${panday} ${pandaz}" rpy="0 0 ${pi/2}"/>
+  <!-- <xacro:panda_arm connected_to="table" xyz="${pandax} ${panday} ${pandaz}" rpy="0 0 ${pi/2}"/> -->
+  <xacro:panda_arm connected_to="table" xyz="${pandax} ${panday} ${pandaz}" rpy="0 0 0"/>
   <xacro:hand_fingers_fixed ns="panda" rpy="0 0 ${-pi/4}" connected_to="panda_link8" q_fingers="0.02"/>
   <xacro:include filename="../mug.xacro"/>

File: urdf/roahm/sphere_col/table_panda_arm_hand_fingers_fixed.urdf (robot description, URDF)
Before this commit: robot panda, 14 links, 13 joints
Joints:
- joint panda_joint_table: origin xyz=0 0 0 rpy=0 0 1.57079632679 -> xyz=0 0 0 rpy=0 0 0

File: urdf/roahm/sphere_col/table_panda_arm_hand_fingers_fixed.urdf.xacro (robot description, xacro)
@@ -5,5 +5,6 @@
   <xacro:include filename="panda_arm.xacro"/>
   <xacro:include filename="hand_fingers_fixed.xacro"/>
-  <xacro:panda_arm connected_to="table" xyz="${pandax} ${panday} ${pandaz}" rpy="0 0 ${pi/2}"/>
+  <!-- <xacro:panda_arm connected_to="table" xyz="${pandax} ${panday} ${pandaz}" rpy="0 0 ${pi/2}"/> -->
+  <xacro:panda_arm connected_to="table" xyz="${pandax} ${panday} ${pandaz}" rpy="0 0 0"/>
   <xacro:hand_fingers_fixed ns="panda" rpy="0 0 ${-pi/4}" connected_to="panda_link8" q_fingers="0.02"/>
 </robot>

File: urdf/roahm/sphere_vis/table_mug_panda_arm_hand_fingers_fixed.urdf (robot description, URDF)
Before this commit: robot panda, 16 links, 15 joints
Joints:
- joint panda_joint_table: origin xyz=0 0 0 rpy=0 0 1.57079632679 -> xyz=0 0 0 rpy=0 0 0

File: urdf/roahm/sphere_vis/table_panda_arm_hand_fingers_fixed.urdf (robot description, URDF)
Before this commit: robot panda, 14 links, 13 joints
Joints:
- joint panda_joint_table: origin xyz=0 0 0 rpy=0 0 1.57079632679 -> xyz=0 0 0 rpy=0 0 0

File: urdf/roahm/table.xacro (robot description, xacro)
@@ -34,5 +34,6 @@
     <visual>
       <!-- <origin xyz="${pandax} ${-pandamounty/2} ${-pandamountz/2+pandamountzoffset}" rpy="0 0 0"/> -->
-      <origin xyz="${pandax} ${panday} ${-pandamountz+pandamountzoffset}" rpy="0 0 ${-pi/2}"/>
+      <!-- <origin xyz="${pandax} ${panday} ${-pandamountz+pandamountzoffset}" rpy="0 0 ${-pi/2}"/>     -->
+      <origin xyz="${pandax} ${panday} ${-pandamountz+pandamountzoffset}" rpy="0 0 0"/>
       <geometry>
         <box size="${pandamountx} ${pandamounty} ${pandamountz}"/>

File: urdf/roahm/table_mug_panda_arm_hand_fingers_fixed.urdf (robot description, URDF)
Before this commit: robot panda, 16 links, 15 joints
Joints:
- joint panda_joint_table: origin xyz=0 0 0 rpy=0 0 1.57079632679 -> xyz=0 0 0 rpy=0 0 0

File: urdf/roahm/table_mug_panda_arm_hand_fingers_fixed.urdf.xacro (robot description, xacro)
@@ -4,5 +4,7 @@
   <xacro:include filename="panda_arm.xacro"/>
   <xacro:include filename="hand_fingers_fixed.xacro"/>
-  <xacro:panda_arm connected_to="table" xyz="${pandax} ${panday} ${pandaz}" rpy="0 0 ${pi/2}"/>
+  <!-- <xacro:panda_arm connected_to="table" xyz="${pandax} ${panday} ${pandaz}" rpy="0 0 ${pi/2}"/> -->
+  <xacro:panda_arm connected_to="table" xyz="${pandax} ${panday} ${pandaz}" rpy="0 0 0"/>
+  <!-- <xacro:panda_arm connected_to="table" xyz="${pandax} ${panday} ${pandaz}" rpy="0 0 ${-pi/2}"/> -->
   <xacro:hand_fingers_fixed ns="panda" rpy="0 0 ${-pi/4}" connected_to="panda_link8" q_fingers="0.02"/>
   <xacro:include filename="mug.xacro"/>

File: urdf/roahm/table_panda_arm_hand_fingers_fixed.urdf (robot description, URDF)
Before this commit: robot panda, 14 links, 13 joints
Joints:
- joint panda_joint_table: origin xyz=0 0 0 rpy=0 0 1.57079632679 -> xyz=0 0 0 rpy=0 0 0

File: urdf/roahm/table_panda_arm_hand_fingers_fixed.urdf.xacro (robot description, xacro)
@@ -4,5 +4,6 @@
   <xacro:include filename="panda_arm.xacro"/>
   <xacro:include filename="hand_fingers_fixed.xacro"/>
-  <xacro:panda_arm connected_to="table" xyz="${pandax} ${panday} ${pandaz}" rpy="0 0 ${pi/2}"/>
+  <!-- <xacro:panda_arm connected_to="table" xyz="${pandax} ${panday} ${pandaz}" rpy="0 0 ${pi/2}"/> -->
+  <xacro:panda_arm connected_to="table" xyz="${pandax} ${panday} ${pandaz}" rpy="0 0 0"/>
   <xacro:hand_fingers_fixed ns="panda" rpy="0 0 ${-pi/4}" connected_to="panda_link8" q_fingers="0.02"/>
 </robot>
